File: em_powerstage/Project Lab 4.kicad_sch (KiCad schematic)
At the start: 43 parts, among them J1 10 PIN ATX, J2 Conn_01x01, J3 Conn_01x01, Q4 NPN, Q5 NMOS, U3 MIC5219-5.0YMM

Commit message: updated power stage board
Parts:
- removed J1: 10 PIN ATX, symbol Connector_Generic:Conn_02x05_Counter_Clockwise
- removed J2, J3: Conn_01x01, symbol Connector_Generic:Conn_01x01
- removed OC1, OC2, OC3: FOD817A, Package_DIP_AKL:DIP-4_W7.62mm_LongPads, symbol PCM_Optocoupler_AKL:FOD817A
- removed Q4: NPN, symbol Device:Q_NPN_BCE
- removed Q5: NMOS, symbol PCM_Transistor_MOSFET_AKL:Q_NMOS-D_Generic_GDS
- removed R16: 100k, symbol Device:R_Small
- removed R17, R18, R19, R20, R22: 1k, symbol Device:R_Small
- removed R21: 100, symbol Device:R_Small
- removed U2, U5: ~, PCM_Package_SO_AKL:QSOP-16_3.9x4.9mm_P0.635mm, symbol HAVENS_Lib:ADUM3195
- added C34: 0.1u, Capacitor_SMD:C_1206_3216Metric_Pad1.33x1.80mm_HandSolder, symbol Device:C_Small
- added D2, D5: LED, LED_SMD:LED_1206_3216Metric_Pad1.42x1.75mm_HandSolder, symbol Device:LED
- added H1: +TWEEZERS, MountingHole:MountingHole_4.3mm_M4_Pad, symbol Mechanical:MountingHole_Pad
- added H2: -TWEEZERS, MountingHole:MountingHole_4.3mm_M4_Pad, symbol Mechanical:MountingHole_Pad
- added H3, H4, H5, H6: MountingHole, MountingHole:MountingHole_4mm, symbol Mechanical:MountingHole
- added H7: Bus Bar, HAVENS_Lib:busbar_28mmX155mm, symbol Mechanical:MountingHole_Pad
- added H8: Bus Bar, HAVENS_Lib:busbar_35mm_18mm, symbol Mechanical:MountingHole_Pad
- added J2: 10 PIN ATX, Connector_Molex:Molex_Mini-Fit_Jr_5566-10A_2x05_P4.20mm_Vertical, symbol Connector_Generic:Conn_02x05_Top_Bottom
- added J4: Conn_02x08_Odd_Even, Connector_PinHeader_2.54mm:PinHeader_2x08_P2.54mm_Vertical, symbol Connector_Generic:Conn_02x08_Odd_Even
- added L1: 47n, Inductor_SMD:L_1206_3216Metric_Pad1.22x1.90mm_HandSolder, symbol Device:L_Small
- added OC1, OC4: VO617A, PCM_Package_DIP_AKL:DIP-4_W7.62mm_LongPads, symbol PCM_Optocoupler_AKL:VO617A
- added R23: 1k, Resistor_SMD:R_0805_2012Metric_Pad1.20x1.40mm_HandSolder, symbol Device:R_Small
- added R24: R_Shunt, HAVENS_Lib:CSM2F6918L050J21, symbol Device:R_Shunt
- added SW1, SW2: SW_SPDT, Button_Switch_THT:SW_E-Switch_EG1271_SPDT, symbol Switch:SW_SPDT
- added TH1, TH2: 10k@25c, Resistor_SMD:R_0402_1005Metric_Pad0.72x0.64mm_HandSolder, symbol Device:Thermistor
- added U2: ISO7341C, Package_SO:SOIC-16W_7.5x10.3mm_P1.27mm, symbol Isolator:ISO7341C
- added U5: ADC104S051, PCM_Package_SO_AKL:MSOP-10-1EP_3x3mm_P0.5mm_EP1.73x1.98mm, symbol HAVENS_Lib:ADC104S051
- added U6: TLV272CS, PCM_Package_SO_AKL:SO-8_3.9x4.9mm_P1.27mm, symbol PCM_Amplifier_Operational_AKL:TLV272CS
- C1, C2, C23, C27, C28, C30, C31, C32, C33: footprint (none) -> Capacitor_SMD:C_1206_3216Metric_Pad1.33x1.80mm_HandSolder
- C29: footprint (none) -> Capacitor_THT:C_Disc_D8.0mm_W2.5mm_P5.00mm
- R1: footprint (none) -> HAVENS_Lib:CSS4J4026RL500F
- R10, R11, R12, R14, R15, R6, R7, R9: footprint (none) -> Resistor_SMD:R_0805_2012Metric_Pad1.20x1.40mm_HandSolder
- R13: value 10k -> 1k; footprint (none) -> Resistor_SMD:R_0805_2012Metric_Pad1.20x1.40mm_HandSolder
- R3: value 0 -> 1k; footprint (none) -> Resistor_SMD:R_0805_2012Metric_Pad1.20x1.40mm_HandSolder
- R4: value 0 -> 470; footprint (none) -> Resistor_SMD:R_0805_2012Metric_Pad1.20x1.40mm_HandSolder
- R8: footprint (none) -> Resistor_THT:R_Axial_DIN0207_L6.3mm_D2.5mm_P15.24mm_Horizontal
Connections:
- net power_stage/DISCHARGE is gone; now on net GNDPWR: R13.2
- net +12V: now also D2.2 (A), J2.10 (Pin_10), OC4.4; no longer R12.1, R13.1
- net +13.8V: now also J2.5 (Pin_5)
- net +40V: now also H7.1, J2.1 (Pin_1), R24.1
- net +5V: now also C31.1, C32.1, C34.1, D5.2 (A), L1.2, SW1.3 (C), SW2.3 (C), TH1.1, TH2.1, U2.10 (EN2), U2.16 (VCC2), U6.8 (V+); no longer C2.1, C33.1
- net +5V_ISO: now also C33.1, J4.1 (Pin_1), J4.2 (Pin_2), J4.5 (Pin_5), J4.6 (Pin_6), U2.1 (VCC1), U2.7 (EN1); no longer C31.1, C32.1
- net +RS: now also R24.2
- net -13.8V: now also J2.3 (Pin_3)
- net -RS: now also R24.3
- net DISCHARGE: now also R12.1, OC4.3; no longer R11.1
- net GAIN1: now also SW1.2 (B); no longer R3.1
- net GAIN2: now also SW2.2 (B); no longer R4.1
- net GND: now also C33.2, J4.3 (Pin_3), J4.4 (Pin_4), J4.7 (Pin_7), J4.8 (Pin_8), OC1.2, OC4.2, U2.2 (GND1), U2.8 (GND1); no longer C31.2, C32.2
- net GNDPWR: now also C31.2, C32.2, R12.2, C34.2, H2.1, J2.2 (Pin_2), J2.4 (Pin_4), J2.6 (Pin_6), J2.7 (Pin_7), J2.9 (Pin_9), OC1.3, R23.2, SW1.1 (A), SW2.1 (A), U2.15 (GND2), U2.9 (GND2), U5.3 (GND), U6.4 (V-); no longer C33.2
- net HV_EN: now also J4.13 (Pin_13)
- net HV_RELAY: now also J2.8 (Pin_8), OC1.4
- net power_stage/+TWEEZER: now also H1.1
- net ~BLEED: now also J4.11 (Pin_11)
- net +v_sens: now reaches R10.2, R9.2
- net +v_sens: now also U6.5 (+)
- net at R11.2: now also OC4.1
- net at R15.2: now also OC1.1
- net -shunt renamed -SHUNT
- net -SHUNT: now also H8.1, R24.4
- net cur_sense renamed +i_sens
- net +i_sens: now also U6.3 (+)
- new net: U2.14 (OUTA), U5.1 (~CS)
- new net: U2.13 (OUTB), U5.10 (SCLK)
- new net: C2.1, L1.1, U5.2 (VCCA)
- new net: U2.12 (OUTC), U5.8 (DIN)
- new net: U2.11 (IND), U5.9 (DOUT)
- new net: D2.1 (K), R3.1
- new net: D5.1 (K), R4.1
- new net I_SENS: U5.4 (IN4), U6.1, U6.2 (-)
- new net MISO: J4.16 (Pin_16), U2.6 (OUTD)
- new net MOSI: J4.14 (Pin_14), U2.5 (INC)
- new net SCLK: J4.12 (Pin_12), U2.4 (INB)
- new net THERM1: R13.1, TH1.2, U5.6 (IN2)
- new net THERM2: R23.1, TH2.2, U5.7 (IN1)
- new net TRIG: J4.15 (Pin_15), R11.1
- new net V_SENS: U5.5 (IN3), U6.6 (-), U6.7
- new net ~CS: J4.10 (Pin_10), U2.3 (INA)
- no-connect marks 5 -> 2
Other:
- sheet cap_bank ports: added ~BLEED; removed none
- sheet power_stage ports: added +CAP; removed +12V
- note added: "< 100mA"
- note added: "Av = 10 | 0 0 Av = 20 | 1 0 Av = 50 | 0 1 Av = 100 | 1 1"
- note added: "Av=10"
- note added: "NTCGS103JX103DT7"
- note added: "must pull 'HV_RELAY' low to enable 40V supply"
- note added: "need 10 pin atx footprint"
- note removed: ">1W"
- note removed: "todo list: pinout for mcu, footprint for caps, footprint for rest of parts"
- moved on the sheet: C1, R11, R6, R7, U1
