File: em_powerstage/power_stage.kicad_sch (KiCad schematic)
At the start: 12 parts, among them IC1 LTC7001EMSE#TRPBF, Q1 IPTG007N06NM5, Q2 IPTG007N06NM5, Q3 IPTG007N06NM5

Commit message: updated power stage board
Parts:
- C24, C25: footprint (none) -> Capacitor_SMD:C_1206_3216Metric_Pad1.33x1.80mm_HandSolder
- C26: footprint (none) -> Capacitor_SMD:C_0805_2012Metric_Pad1.18x1.45mm_HandSolder
- IC1: footprint SOP50P490X110-11N -> HAVENS_Lib:SOP50P490X110-11N
- Q1, Q2, Q3: footprint Package_TO_SOT_SMD:Infineon_PG-HSOF-8-1_ThermalVias -> HAVENS_Lib:HSOG_8-3
- R2, R5: footprint (none) -> Resistor_SMD:R_0805_2012Metric_Pad1.20x1.40mm_HandSolder
Connections:
- net -SHUNT: no longer D4.3 (K)
- net gate: now reaches C26.1, IC1.6 (TGDN), Q1.1 (G), Q2.1 (G), Q3.1 (G), R5.2
- new net +CAP: D4.3 (K)
Changed lines of the file:
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@@
-	)
-	(junction
-		(at 186.69 62.23)
-		(diameter 0)
-		(color 0 0 0 0)
 	)
 	(junction
@@
 	(wire
 		(pts
-			(xy 171.45 72.39) (xy 171.45 62.23)
+			(xy 171.45 72.39) (xy 171.45 57.15)
 		)
 		(stroke
@@
 	(wire
 		(pts
-			(xy 171.45 62.23) (xy 186.69 62.23)
-		)
-		(stroke
-			(width 0)
-			(type default)
-		)
-	)
-	(wire
-		(pts
 			(xy 127 110.49) (xy 134.62 110.49)
 		)
@@
 	(wire
 		(pts
-			(xy 186.69 62.23) (xy 186.69 96.52)
+			(xy 186.69 57.15) (xy 186.69 96.52)
 		)
 		(stroke
@@
 	(wire
 		(pts
-			(xy 186.69 57.15) (xy 186.69 62.23)
-		)
-		(stroke
-			(width 0)
-			(type default)
-		)
-	)
-	(wire
-		(pts
 			(xy 106.68 81.28) (xy 106.68 80.01)
 		)
@@
 			(width 0)
 			(type default)
+		)
+	)
+	(label "gate"
+		(at 154.94 102.87 0)
+		(fields_autoplaced yes)
+		(effects
+			(font
+				(size 1.27 1.27)
+			)
+			(justify left bottom)
 		)
 	)
@@
 		)
 	)
-	(hierarchical_label "DISCHARGE"
+	(hierarchical_label "+CAP"
 		(shape bidirectional)
-		(at 96.52 102.87 180)
+		(at 171.45 57.15 90)
 		(fields_autoplaced yes)
 		(effects
 			(font
 				(size 1.27 1.27)
-				(bold yes)
-			)
-			(justify right)
-		)
-	)
-	(hierarchical_label "+12V"
+			)
+			(justify left)
+		)
+	)
+	(hierarchical_label "DISCHARGE"
 		(shape bidirectional)
-		(at 72.39 99.06 180)
+		(at 96.52 102.87 180)
 		(fields_autoplaced yes)
 		(effects
@@
 		)
 		(instances
-			(project ""
+			(project "Project Lab 4"
 				(path "/f55c1fef-06fc-4e91-9a1e-7c26aa5a1e26/6af4c692-356b-4b64-a980-f9d4755c173b"
 					(reference "#PWR03")
@@
 			)
 		)
-		(property "Footprint" ""
+		(property "Footprint" "Capacitor_SMD:C_1206_3216Metric_Pad1.33x1.80mm_HandSolder"
 			(at 134.62 97.79 0)
 			(effects
@@
 			)
 		)
-		(property "Footprint" "Package_TO_SOT_SMD:Infineon_PG-HSOF-8-1_ThermalVias"
+		(property "Footprint" "HAVENS_Lib:HSOG_8-3"
 			(at 204.47 104.775 0)
 			(effects
@@
 			)
 		)
-		(property "Footprint" ""
+		(property "Footprint" "Resistor_SMD:R_0805_2012Metric_Pad1.20x1.40mm_HandSolder"
 			(at 149.86 121.92 0)
 			(effects
@@
 		)
 		(instances
-			(project ""
+			(project "Project Lab 4"
 				(path "/f55c1fef-06fc-4e91-9a1e-7c26aa5a1e26/6af4c692-356b-4b64-a980-f9d4755c173b"
 					(reference "R2")
@@
 			)
 		)
-		(property "Footprint" "SOP50P490X110-11N"
+		(property "Footprint" "HAVENS_Lib:SOP50P490X110-11N"
 			(at 123.19 188.9 0)
 			(effects
@@
 			)
 		)
-		(property "Footprint" "Package_TO_SOT_SMD:Infineon_PG-HSOF-8-1_ThermalVias"
+		(property "Footprint" "HAVENS_Lib:HSOG_8-3"
 			(at 189.23 104.775 0)
 			(effects
@@
 	)
 	(symbol
+		(lib_id "power:+12V")
+		(at 72.39 99.06 0)
+		(unit 1)
+		(exclude_from_sim no)
+		(in_bom yes)
+		(on_board yes)
+		(dnp no)
+		(property "Reference" "#PWR017"
+			(at 72.39 102.87 0)
+			(effects
+				(font
+					(size 1.27 1.27)
+				)
+				(hide yes)
+			)
+		)
+		(property "Value" "+12V"
+			(at 72.39 95.25 0)
+			(effects
+				(font
+					(size 1.27 1.27)
+				)
+			)
+		)
+		(property "Footprint" ""
+			(at 72.39 99.06 0)
+			(effects
+				(font
+					(size 1.27 1.27)
+				)
+				(hide yes)
+			)
+		)
+		(property "Datasheet" ""
+			(at 72.39 99.06 0)
+			(effects
+				(font
+					(size 1.27 1.27)
+				)
+				(hide yes)
+			)
+		)
+		(property "Description" "Power symbol creates a global label with name \"+12V\""
+			(at 72.39 99.06 0)
+			(effects
+				(font
+					(size 1.27 1.27)
+				)
+				(hide yes)
+			)
+		)
+		(pin "1"
+		)
+		(instances
+			(project "Project Lab 4"
+				(path "/f55c1fef-06fc-4e91-9a1e-7c26aa5a1e26/6af4c692-356b-4b64-a980-f9d4755c173b"
+					(reference "#PWR017")
+					(unit 1)
+				)
+			)
+		)
+	)
+	(symbol
 		(lib_id "Transistor_FET:IPT015N10N5")
 		(at 168.91 102.87 0)
@@
 			)
 		)
-		(property "Footprint" "Package_TO_SOT_SMD:Infineon_PG-HSOF-8-1_ThermalVias"
+		(property "Footprint" "HAVENS_Lib:HSOG_8-3"
 			(at 173.99 104.775 0)
 			(effects
@@
 			)
 		)
-		(property "Footprint" ""
+		(property "Footprint" "Capacitor_SMD:C_0805_2012Metric_Pad1.18x1.45mm_HandSolder"
 			(at 149.86 114.3 0)
 			(effects
@@
 		)
 		(instances
-			(project ""
+			(project "Project Lab 4"
 				(path "/f55c1fef-06fc-4e91-9a1e-7c26aa5a1e26/6af4c692-356b-4b64-a980-f9d4755c173b"
 					(reference "C26")
@@
 			)
 		)
-		(property "Footprint" ""
+		(property "Footprint" "Resistor_SMD:R_0805_2012Metric_Pad1.20x1.40mm_HandSolder"
 			(at 142.24 101.6 0)
 			(effects
@@
 		)
 		(instances
-			(project ""
+			(project "Project Lab 4"
 				(path "/f55c1fef-06fc-4e91-9a1e-7c26aa5a1e26/6af4c692-356b-4b64-a980-f9d4755c173b"
 					(reference "R5")
@@
 			)
 		)
-		(property "Footprint" ""
+		(property "Footprint" "Capacitor_SMD:C_1206_3216Metric_Pad1.33x1.80mm_HandSolder"
 			(at 74.93 104.14 0)
 			(effects
@@
 		)
 		(instances
-			(project ""
+			(project "Project Lab 4"
 				(path "/f55c1fef-06fc-4e91-9a1e-7c26aa5a1e26/6af4c692-356b-4b64-a980-f9d4755c173b"
 					(reference "C24")
@@
 		)
 		(instances
-			(project ""
+			(project "Project Lab 4"
 				(path "/f55c1fef-06fc-4e91-9a1e-7c26aa5a1e26/6af4c692-356b-4b64-a980-f9d4755c173b"
 					(reference "D4")
