File: em_powerstage/Project Lab 4.kicad_pcb (KiCad board)
At the start: 4 copper layers, 33 parts, among them IC1 LTC7001MPMSE#PBF, Q1 IPTG007N06NM5ATMA1, Q2 IPTG007N06NM5ATMA1, Q3 IPTG007N06NM5ATMA1

Commit message: updated power stage board
Parts:
- added C22: 33m, HAVENS_Lib:CAPPRD1000W190D3550H8200, F.Cu at (326.5, 188.8)
- added C25: 1u, Capacitor_SMD:C_1206_3216Metric_Pad1.33x1.80mm_HandSolder, F.Cu at (422.2, 0.61)
- added C26: 47n, Capacitor_SMD:C_0805_2012Metric_Pad1.18x1.45mm_HandSolder, F.Cu at (417.2, 0.70)
- added C27: 0.1u, Capacitor_SMD:C_1206_3216Metric_Pad1.33x1.80mm_HandSolder, F.Cu at (355.6, 12.8)
- added C28: 0.1u, Capacitor_SMD:C_1206_3216Metric_Pad1.33x1.80mm_HandSolder, F.Cu at (373.9, -19.8)
- added C29: Y, Capacitor_THT:C_Disc_D8.0mm_W2.5mm_P5.00mm, F.Cu at (351.8, -20.9)
- added C30: 0.1u, Capacitor_SMD:C_1206_3216Metric_Pad1.33x1.80mm_HandSolder, F.Cu at (364.8, -33.2)
- added C31: 0.1u, Capacitor_SMD:C_1206_3216Metric_Pad1.33x1.80mm_HandSolder, F.Cu at (437.7, -4.70)
- added C32: 0.1u, Capacitor_SMD:C_1206_3216Metric_Pad1.33x1.80mm_HandSolder, F.Cu at (451.4, 3.60)
- added C33: 0.1u, Capacitor_SMD:C_1206_3216Metric_Pad1.33x1.80mm_HandSolder, F.Cu at (451.3, -26.2)
- added C34: 0.1u, Capacitor_SMD:C_1206_3216Metric_Pad1.33x1.80mm_HandSolder, F.Cu at (451.3, -19.2)
- added D3: V8P10, Package_TO_SOT_SMD:TO-277A, F.Cu at (371.6, 2.55)
- added D4: V8P10, Package_TO_SOT_SMD:TO-277A, F.Cu at (408.4, 38.0)
- added D5: LED, LED_SMD:LED_1206_3216Metric_Pad1.42x1.75mm_HandSolder, F.Cu at (325.9, 2.30)
- added H1: +TWEEZERS, MountingHole:MountingHole_4.3mm_M4_Pad, F.Cu at (393.8, -7.00)
- added H2: -TWEEZERS, MountingHole:MountingHole_4.3mm_M4_Pad, F.Cu at (393.8, -17.6)
- added H3: MountingHole, MountingHole:MountingHole_4mm, F.Cu at (333.0, -35.0)
- added H4: MountingHole, MountingHole:MountingHole_4mm, F.Cu at (455.0, -35.0)
- added H5: MountingHole, MountingHole:MountingHole_4mm, F.Cu at (333.0, 218.8)
- added H6: MountingHole, MountingHole:MountingHole_4mm, F.Cu at (455.0, 218.8)
- added H7: Bus Bar, HAVENS_Lib:busbar_28mmX155mm, F.Cu at (393.8, 148.6)
- added H8: Bus Bar, HAVENS_Lib:busbar_35mm_18mm, F.Cu at (394.0, 22.5)
- added J2: 10 PIN ATX, Connector_Molex:Molex_Mini-Fit_Jr_5566-10A_2x05_P4.20mm_Vertical, F.Cu at (340.6, 16.9)
- added J4: Conn_02x08_Odd_Even, Connector_PinHeader_2.54mm:PinHeader_2x08_P2.54mm_Vertical, F.Cu at (384.9, -38.3)
- added L1: 47n, Inductor_SMD:L_1206_3216Metric_Pad1.22x1.90mm_HandSolder, F.Cu at (439.0, -0.90)
- added OC1: VO617A, PCM_Package_DIP_AKL:DIP-4_W7.62mm_LongPads, F.Cu at (346.7, -27.0)
- added OC2: VO617A, PCM_Package_DIP_AKL:DIP-4_W7.62mm_LongPads, F.Cu at (430.5, -26.6)
- added OC4: VO617A, PCM_Package_DIP_AKL:DIP-4_W7.62mm_LongPads, F.Cu at (423.1, -26.6)
- added Q5: NMOS, Package_TO_SOT_SMD:SOT-23-3, F.Cu at (430.2, 13.2)
- added R10: 47k, Resistor_SMD:R_0805_2012Metric_Pad1.20x1.40mm_HandSolder, F.Cu at (462.8, 24.2)
- added R11: 100, Resistor_SMD:R_0805_2012Metric_Pad1.20x1.40mm_HandSolder, F.Cu at (423.2, -31.8)
- added R12: 10k, Resistor_SMD:R_0805_2012Metric_Pad1.20x1.40mm_HandSolder, F.Cu at (420.4, -14.0)
- added R13: 1k, Resistor_SMD:R_0805_2012Metric_Pad1.20x1.40mm_HandSolder, F.Cu at (448.2, -3.73)
- added R14: 10k, Resistor_SMD:R_0805_2012Metric_Pad1.20x1.40mm_HandSolder, F.Cu at (347.6, -16.1)
- added R15: 100, Resistor_SMD:R_0805_2012Metric_Pad1.20x1.40mm_HandSolder, F.Cu at (346.6, -31.4)
- added R16: 100, Resistor_SMD:R_0805_2012Metric_Pad1.20x1.40mm_HandSolder, F.Cu at (430.8, -31.8)
- added R17: 100k, Resistor_SMD:R_0805_2012Metric_Pad1.20x1.40mm_HandSolder, F.Cu at (430.2, 22.4)
- added R18: 1k, Resistor_SMD:R_1218_3246Metric_Pad1.22x4.75mm_HandSolder, F.Cu at (450.0, 18.0)
- added R19: 1k, Resistor_SMD:R_1218_3246Metric_Pad1.22x4.75mm_HandSolder, F.Cu at (455.5, 18.0)
- added R20: 1k, Resistor_SMD:R_1218_3246Metric_Pad1.22x4.75mm_HandSolder, F.Cu at (444.5, 18.0)
- added R21: 1k, Resistor_SMD:R_1218_3246Metric_Pad1.22x4.75mm_HandSolder, F.Cu at (439.0, 18.0)
- added R22: 1k, Resistor_SMD:R_1218_3246Metric_Pad1.22x4.75mm_HandSolder, F.Cu at (433.5, 18.0)
- added R23: 1k, Resistor_SMD:R_0805_2012Metric_Pad1.20x1.40mm_HandSolder, F.Cu at (451.4, -3.73)
- added R24: R_Shunt, HAVENS_Lib:CSM2F6918L050J21, F.Cu at (393.8, 54.7)
- added R5: 1k, Resistor_SMD:R_0805_2012Metric_Pad1.20x1.40mm_HandSolder, F.Cu at (419.5, 0.70)
- added R6: 0, Resistor_SMD:R_0805_2012Metric_Pad1.20x1.40mm_HandSolder, F.Cu at (359.0, 31.7)
- added R7: 0, Resistor_SMD:R_0805_2012Metric_Pad1.20x1.40mm_HandSolder, F.Cu at (359.0, 29.5)
- added R8: 1Meg, Resistor_THT:R_Axial_DIN0207_L6.3mm_D2.5mm_P15.24mm_Horizontal, F.Cu at (355.6, -15.6)
- added R9: 470k, Resistor_SMD:R_0805_2012Metric_Pad1.20x1.40mm_HandSolder, F.Cu at (458.2, 24.2)
- added SW1: SW_SPDT, Button_Switch_THT:SW_E-Switch_EG1271_SPDT, F.Cu at (328.9, -17.9)
- added SW2: SW_SPDT, Button_Switch_THT:SW_E-Switch_EG1271_SPDT, F.Cu at (336.9, -17.9)
- added TH1: 10k@25c, Resistor_SMD:R_0402_1005Metric_Pad0.72x0.64mm_HandSolder, B.Cu at (394.0, 14.3)
- added TH2: 10k@25c, Resistor_SMD:R_0402_1005Metric_Pad0.72x0.64mm_HandSolder, B.Cu at (393.8, 168.3)
- added U1: ~, HAVENS_Lib:TDFN-10-SMD, F.Cu at (367.2, 30.5)
- added U2: ISO7341C, Package_SO:SOIC-16W_7.5x10.3mm_P1.27mm, F.Cu at (443.8, -22.8)
- added U3: MIC5219-5.0YMM, Package_SO:MSOP-8_3x3mm_P0.65mm, F.Cu at (356.0, 17.8)
- added U4: ~, HAVENS_Lib:1769405241, F.Cu at (364.8, -22.6)
- added U5: ADC104S051, PCM_Package_SO_AKL:MSOP-10-1EP_3x3mm_P0.5mm_EP1.73x1.98mm, F.Cu at (444.5, -2.56)
- added U6: TLV272CS, PCM_Package_SO_AKL:SO-8_3.9x4.9mm_P1.27mm, F.Cu at (444.5, 5.40)
- C1: value 47n -> 0.1u; footprint Capacitor_SMD:C_0805_2012Metric -> Capacitor_SMD:C_1206_3216Metric_Pad1.33x1.80mm_HandSolder
- C10, C11, C12, C13, C14, C15, C16, C17, C18, C19, C20, C21, C3, C4, C5, C6, C7, C8, C9: footprint Capacitor_THT:CP_Radial_D22.0mm_P10.00mm_SnapIn -> HAVENS_Lib:CAPPRD1000W190D3550H8200
- C2: value .1u -> 0.1u; footprint Capacitor_SMD:C_0805_2012Metric -> Capacitor_SMD:C_1206_3216Metric_Pad1.33x1.80mm_HandSolder
- C23: value 33m -> 0.1u; footprint Capacitor_THT:CP_Radial_D22.0mm_P10.00mm_SnapIn -> Capacitor_SMD:C_1206_3216Metric_Pad1.33x1.80mm_HandSolder
- C24: value .47u -> 0.1u; footprint Capacitor_SMD:C_0805_2012Metric -> Capacitor_SMD:C_1206_3216Metric_Pad1.33x1.80mm_HandSolder
- D1: value D -> D_AAK; footprint Diode_SMD:D_0805_2012Metric -> Package_TO_SOT_SMD:SOT-23-3
- D2: value D -> LED; footprint Diode_SMD:D_0805_2012Metric -> LED_SMD:LED_1206_3216Metric_Pad1.42x1.75mm_HandSolder
- IC1: value LTC7001MPMSE#PBF -> LTC7001EMSE#TRPBF; footprint KiCad:SOP50P490X110-11N -> HAVENS_Lib:SOP50P490X110-11N
- Q1, Q2, Q3: value IPTG007N06NM5ATMA1 -> IPTG007N06NM5; footprint KiCad_iptg:IPTG007N06NM5ATMA1 -> HAVENS_Lib:HSOG_8-3
- R1: value 1k -> R_Shunt; footprint Resistor_SMD:R_0805_2012Metric -> HAVENS_Lib:CSS4J4026RL500F
- R2: footprint Resistor_SMD:R_0805_2012Metric -> Resistor_SMD:R_0805_2012Metric_Pad1.20x1.40mm_HandSolder
- R3: value 590k -> 1k; footprint Resistor_SMD:R_0805_2012Metric -> Resistor_SMD:R_0805_2012Metric_Pad1.20x1.40mm_HandSolder
- R4: value 12k -> 470; footprint Resistor_SMD:R_0805_2012Metric -> Resistor_SMD:R_0805_2012Metric_Pad1.20x1.40mm_HandSolder
- moved C16 424.2 mm to (461.0, 78.7)
- moved C4 417.4 mm to (461.0, 188.8)
- moved C8 388.1 mm to (461.0, 152.1), turned to -90 degrees
- moved C7 383.8 mm to (427.5, 169.7), turned to -90 degrees
- moved C20 375.8 mm to (461.0, 42.0), turned to -90 degrees
- moved C3 368.8 mm to (427.5, 206.4)
- moved C19 367.2 mm to (427.5, 59.6), turned to -90 degrees
- moved C15 366.5 mm to (427.5, 96.3)
- moved C12 355.0 mm to (461.0, 115.4)
- moved C5 351.0 mm to (360.0, 206.4)
- moved C17 329.0 mm to (360.0, 96.3), turned to -90 degrees
- moved C11 301.2 mm to (427.5, 133.0)
- moved C6 289.4 mm to (326.5, 42.0), turned to -90 degrees
- moved C9 275.6 mm to (360.0, 169.7), turned to -90 degrees
- moved C2 273.5 mm to (437.7, 2.90)
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Connections:
- C1 pad 1: Net-(IC1-TGDN) -> +5V
- C1 pad 2: Net-(C1-Pad2) -> GNDPWR
- C10 pad 2: GND -> GNDPWR
- C11 pad 2: GND -> GNDPWR
- C12 pad 2: GND -> GNDPWR
- C13 pad 2: GND -> GNDPWR
- C14 pad 2: GND -> GNDPWR
- C15 pad 2: GND -> GNDPWR
- C16 pad 2: GND -> GNDPWR
- C17 pad 2: GND -> GNDPWR
- C18 pad 2: GND -> GNDPWR
- C19 pad 2: GND -> GNDPWR
- C2 pad 1: Net-(IC1-TS) -> Net-(U5-VCCA)
- C2 pad 2: Net-(D1-A) -> GNDPWR
- C20 pad 2: GND -> GNDPWR
- C21 pad 2: GND -> GNDPWR
- C23 pad 1: +40V -> +5V
- C23 pad 2: GND -> GNDPWR
- C24 pad 1: GND -> +12V
- C24 pad 2: +40V -> GNDPWR
- C3 pad 2: GND -> GNDPWR
- C4 pad 2: GND -> GNDPWR
- C5 pad 2: GND -> GNDPWR
- C6 pad 2: GND -> GNDPWR
- C7 pad 2: GND -> GNDPWR
- C8 pad 2: GND -> GNDPWR
- C9 pad 2: GND -> GNDPWR
- D1 pad 2: Net-(D1-A) -> +12V
- D2 pad 1: +40V -> Net-(D2-K)
- D2 pad 2: +40V -> +12V
- IC1 pad 11: GND -> GNDPWR
- IC1 pad 3: GND -> GNDPWR
- IC1 pad 4: /Input Signal -> /DISCHARGE
- IC1 pad 5: Net-(IC1-OVLO) -> unconnected-(IC1-OVLO-Pad5)
- IC1 pad 6: Net-(IC1-TGDN) -> /power_stage/gate
- IC1 pad 8: Net-(IC1-TS) -> /power_stage/+TWEEZER
- IC1 pad 9: Net-(D1-A) -> Net-(D1-K)
- Q1 pad 1: Net-(IC1-TGDN) -> /power_stage/gate
- Q1 pad 2: Net-(IC1-TS) -> /power_stage/+TWEEZER
- Q1 pad 3: unconnected-(Q1-S_2-Pad3) -> /-SHUNT
- Q2 pad 1: Net-(IC1-TGDN) -> /power_stage/gate
- Q2 pad 2: Net-(IC1-TS) -> /power_stage/+TWEEZER
- Q2 pad 3: unconnected-(Q2-S_2-Pad3) -> /-SHUNT
- Q3 pad 1: Net-(IC1-TGDN) -> /power_stage/gate
- Q3 pad 2: Net-(IC1-TS) -> /power_stage/+TWEEZER
- Q3 pad 3: unconnected-(Q3-S_2-Pad3) -> /-SHUNT
- R1 pad 1: Net-(IC1-TGUP) -> +40V
- R1 pad 2: Net-(IC1-TGDN) -> /+RS
- R2 pad 1: Net-(C1-Pad2) -> Net-(C26-Pad2)
- R2 pad 2: GND -> GNDPWR
- R3 pad 1: Net-(IC1-OVLO) -> Net-(D2-K)
- R3 pad 2: +40V -> GNDPWR
- R4 pad 1: GND -> Net-(D5-K)
- R4 pad 2: Net-(IC1-OVLO) -> GNDPWR
Routing:
- net +40V: track 531.9 -> 0.00 mm
- net THERM2: track 0.00 -> 221.1 mm, vias 0 -> 1
- net +5V: track 0.00 -> 172.8 mm, vias 0 -> 2
- net /+i_sens: track 0.00 -> 84.3 mm, vias 0 -> 2
- net /GAIN1: track 0.00 -> 69.5 mm, vias 0 -> 1
- net THERM1: track 0.00 -> 67.3 mm, vias 0 -> 1
- net /GAIN2: track 0.00 -> 61.0 mm, vias 0 -> 1
- net /~CS: track 0.00 -> 59.5 mm
- net HV_EN: track 0.00 -> 56.0 mm, vias 0 -> 1
- net /SCLK: track 0.00 -> 55.4 mm
- net /MOSI: track 0.00 -> 51.4 mm
- net /MISO: track 0.00 -> 47.3 mm
- net /cap_bank/bleed_gate: track 0.00 -> 46.6 mm
- net /power_stage/gate: track 0.00 -> 46.4 mm
- net Net-(IC1-TGDN): track 45.5 -> 0.00 mm
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- added copper zone on B.Cu, net +12V
- added copper zone on F.Cu, net +12V
- added copper zone on F.Cu, net +40V
- added copper zone on F.Cu, net +5V
- added copper zone on F.Cu, net +5V_ISO
- added copper zone on B.Cu, net /-SHUNT
- added copper zone on F.Cu, net /-SHUNT
- added copper zone on F.Cu, net /cap_bank/bleed_drain
- added copper zone on F.Cu, net /power_stage/+TWEEZER
- added copper zone on In1.Cu, net GND
- added copper zone on In2.Cu, net GND
- added copper zone on F.Cu, net GNDPWR
- added copper zone on In1.Cu, net GNDPWR
- added copper zone on In2.Cu, net GNDPWR
Other:
- board outline added: 145 x 275 mm
- board text added: "+"
- board text added: "-"
- board text added: "10x | 0 0 20x | 1 0 50x | 0 1 100x | 1 1"
- board text added: "12V"
- board text added: "5V"
- board text added: "GAIN1"
- board text added: "GAIN2"

Commit message: updates
Routing:
- net +12V: track 42.8 -> 47.0 mm
- net Net-(C26-Pad2): track 0.00 -> 2.26 mm
- net GNDPWR: track 10.5 -> 11.2 mm
- net GND: vias 2 -> 5
